File: PCB/V1.0/PnP-Expansion-V1.sch (EAGLE design)
At the start: 62 parts, among them IC1 SP3485EN-L, IC10 FT230XQ, IC11 XR22404CG28TR-F, IC2 SP3485EN-L, IC3 SP3485EN-L, IC4 2SMPP-03, IC5 INA126EA_2K5, IC6 LM358DR2G, IC7 2SMPP-03, IC8 INA126EA_2K5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

Commit message: v1 update
Parts:
- removed AUX-1, AUX-2: (no value), pinhead:PINHD-2X5
Connections:
- removed net AUX_1_A1: AUX-1.2, EXPANSION-1.14
- removed net AUX_1_A2: AUX-1.1, EXPANSION-1.16
- removed net AUX_1_D1: AUX-1.3, EXPANSION-1.12
- removed net AUX_2_A1: AUX-2.2, EXPANSION-2.16
- removed net AUX_2_A2: AUX-2.1, EXPANSION-2.18
- removed net AUX_2_D1: AUX-2.3, EXPANSION-2.14
- removed net MISO: AUX-1.5, AUX-2.5, EXPANSION-1.17
- removed net MOSI: AUX-1.6, AUX-2.6, EXPANSION-1.15
- removed net SCK: AUX-1.4, AUX-2.4, EXPANSION-1.18
- removed net SCL: AUX-1.7, AUX-2.7, EXPANSION-1.13
- removed net SDA: AUX-1.8, AUX-2.8, EXPANSION-1.11
- net +5V: no longer AUX-1.10, AUX-2.10
- net GND: no longer AUX-1.9, AUX-2.9
Other:
- note removed: "AUX"
